File: 1_3/1_3AS/1_3AS.kicad_sch (KiCad schematic)
At the start: 43 parts, among them SW10 SW_SPST, SW11 SW_SPST, SW12 SW_SPST, SW14 SW_SPST, SW15 SW_SPST, SW16 SW_SPST, SW17 SW_SPST, SW18 SW_SPST, SW19 SW_SPST, SW2 SW_SPST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

Commit message: AS add step & gerbers
Parts:
- removed H1: MountingHole, Two:Hole_5.7mm, symbol Two:MountingHole
Changed lines of the file:
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@@
-	)
-	(symbol
-		(lib_id "Two:MountingHole")
-		(at 26.67 110.49 0)
-		(unit 1)
-		(exclude_from_sim no)
-		(in_bom yes)
-		(on_board yes)
-		(dnp no)
-		(fields_autoplaced yes)
-		(property "Reference" "H1"
-			(at 29.21 109.2199 0)
-			(effects
-				(font
-					(size 1.27 1.27)
-				)
-				(justify left)
-			)
-		)
-		(property "Value" "MountingHole"
-			(at 29.21 111.7599 0)
-			(effects
-				(font
-					(size 1.27 1.27)
-				)
-				(justify left)
-			)
-		)
-		(property "Footprint" "Two:Hole_5.7mm"
-			(at 26.67 110.49 0)
-			(effects
-				(font
-					(size 1.27 1.27)
-				)
-				(hide yes)
-			)
-		)
-		(property "Datasheet" "~"
-			(at 26.67 110.49 0)
-			(effects
-				(font
-					(size 1.27 1.27)
-				)
-				(hide yes)
-			)
-		)
-		(property "Description" "Mounting Hole without connection"
-			(at 26.67 110.49 0)
-			(effects
-				(font
-					(size 1.27 1.27)
-				)
-				(hide yes)
-			)
-		)
-		(instances
-			(project "pcb"
-				(path "/1fd8269d-bfbb-4294-b901-abae7a95debd"
-					(reference "H1")
-					(unit 1)
-				)
-			)
-		)
 	)
 	(symbol
