File: 1_3/1_3S/1_3S.kicad_sch (KiCad schematic)
At the start: 49 parts, among them SW1 SW_SPST, SW10 SW_SPST, SW11 SW_SPST, SW12 SW_SPST, SW13 SW_SPST, SW14 SW_SPST, SW15 SW_SPST, SW16 SW_SPST, SW17 SW_SPST, SW18 SW_SPST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

Commit message: 1_3S rebuild
Parts:
- removed D1, D13, D7: D_Small, Two:Diode_TH_SMD_DUAL, symbol Two:D_Small
- removed SW1, SW13, SW7: SW_SPST, Two:KS-27_KS-33_Hotswap_1U_DUAL, symbol Two:SW_SPST
Connections:
- net C0: no longer names the net of U1.1 (A2/0.02_H)
- no-connect marks 4 -> 5
