File: 1_3/1_3/1_3.kicad_pcb (KiCad board)
At the start: 2 copper layers, 137.5 x 91.4 mm, 52 parts, among them SW1 SW_SPST, SW10 SW_SPST, SW11 SW_SPST, SW12 SW_SPST, SW13 SW_SPST, SW14 SW_SPST, SW15 SW_SPST, SW16 SW_SPST, SW17 SW_SPST, SW18 SW_SPST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

Commit message: 1_3 tune
Parts:
- moved D21 0.20 mm to (194.6, 125.0)
- moved D20 0.11 mm to (173.8, 116.4)
Routing:
- net Net-(D19-A): track 18.3 -> 19.4 mm
- net R3: track 128.1 -> 128.8 mm
